File: PCB/psocpcb_v2/psocpcb.kicad_pcb (KiCad board)
At the start: 4 copper layers, 64.8 x 29.8 mm, 49 parts, among them J1 Conn_01x05, J2 Conn_01x02_Pin, J5 Conn_01x04_Pin, J7 Conn_01x06_Pin, Q1 Si2337DS, U2 AP7365-WG-7, U3 AP2331SA-7, U4 SIP32408DNP-T1-GE4, U5 TXS0102DCUR, U6 AP7365-WG-7, U7 CYBLE-416045-02, Y1 ECS-.327-12.5-34B-TR

Commit message: R3
Parts:
- moved J2 0.25 mm to (132.2, 69.8)
Connections:
- A1 pad 11: unconnected-(A1-GPIO17/GEN0-Pad11) -> /GPIO1
- A1 pad 12: unconnected-(A1-GPIO18-Pad12) -> /GPIO2
- A1 pad 13: unconnected-(A1-GPIO27/GEN2-Pad13) -> /SCL
- A1 pad 15: unconnected-(A1-GPIO22/GEN3-Pad15) -> /SDA
- A1 pad 16: unconnected-(A1-GEN4/GPIO23-Pad16) -> /GPIO3
- A1 pad 17: unconnected-(A1-3V3[2]-Pad17) -> /GPIO4
- A1 pad 18: unconnected-(A1-GEN5/GPIO24-Pad18) -> /GPIO5
- A1 pad 19: unconnected-(A1-GPIO10/MOSI-Pad19) -> /GPIO6
- A1 pad 21: unconnected-(A1-GPIO9/MISO-Pad21) -> /GPIO7
- A1 pad 22: unconnected-(A1-GEN/6GPIO25-Pad22) -> /GPIO8
- A1 pad 23: unconnected-(A1-GPIO11/SCLK-Pad23) -> /GPIO9
- A1 pad 24: unconnected-(A1-~{CE0}/GPIO8-Pad24) -> /GPIO10
- A1 pad 26: unconnected-(A1-~{CE1}/~{GPIO7}-Pad26) -> /GPIO11
- A1 pad 27: unconnected-(A1-ID_SD-Pad27) -> /GPIO12
- A1 pad 28: unconnected-(A1-ID_SC-Pad28) -> /GPIO13
- A1 pad 29: unconnected-(A1-GPIO5-Pad29) -> /GPIO14
- A1 pad 31: unconnected-(A1-GPIO6-Pad31) -> /GPIO21
- A1 pad 32: unconnected-(A1-GPIO12-Pad32) -> /GPIO22
- A1 pad 33: unconnected-(A1-GPIO13-Pad33) -> /GPIO20
- A1 pad 35: unconnected-(A1-GPIO19-Pad35) -> /GPIO18
- A1 pad 36: unconnected-(A1-GPIO16-Pad36) -> /GPIO19
- A1 pad 37: unconnected-(A1-GPIO26-Pad37) -> /GPIO16
- A1 pad 38: unconnected-(A1-GPIO20-Pad38) -> /GPIO17
- A1 pad 40: unconnected-(A1-GPIO21-Pad40) -> /GPIO15
- U7 pad 13: unconnected-(U7-P10.0-Pad13) -> /GPIO3
- U7 pad 14: unconnected-(U7-P9.4-Pad14) -> /GPIO4
- U7 pad 16: unconnected-(U7-VREF-Pad16) -> /GPIO5
- U7 pad 19: unconnected-(U7-P9.5-Pad19) -> /GPIO6
- U7 pad 2: unconnected-(U7-P0.5-Pad2) -> /GPIO1
- U7 pad 20: unconnected-(U7-P9.6-Pad20) -> /GPIO7
- U7 pad 21: unconnected-(U7-P9.2-Pad21) -> /GPIO8
- U7 pad 22: unconnected-(U7-P7.2-Pad22) -> /GPIO9
- U7 pad 23: unconnected-(U7-P7.1-Pad23) -> /GPIO10
- U7 pad 24: unconnected-(U7-P6.4-Pad24) -> /GPIO11
- U7 pad 25: unconnected-(U7-P5.4-Pad25) -> /GPIO12
- U7 pad 28: unconnected-(U7-P6.2-Pad28) -> /GPIO13
- U7 pad 29: unconnected-(U7-P6.5-Pad29) -> /GPIO14
- U7 pad 31: unconnected-(U7-P7.7-Pad31) -> /GPIO15
- U7 pad 32: unconnected-(U7-P5.6-Pad32) -> /GPIO16
- U7 pad 34: unconnected-(U7-P12.6-Pad34) -> /GPIO17
- U7 pad 35: unconnected-(U7-P12.7-Pad35) -> /GPIO18
- U7 pad 36: unconnected-(U7-P5.5-Pad36) -> /GPIO19
- U7 pad 37: unconnected-(U7-P5.3-Pad37) -> /GPIO20
- U7 pad 38: unconnected-(U7-P5.2-Pad38) -> /GPIO21
- U7 pad 41: unconnected-(U7-P0.4-Pad41) -> /GPIO22
- U7 pad 9: unconnected-(U7-P9.3-Pad9) -> /GPIO2
Routing:
- net /GPIO2: track 0.00 -> 35.9 mm, vias 0 -> 1
- net /GPIO1: track 0.00 -> 34.8 mm, vias 0 -> 1
- net /GPIO22: track 0.00 -> 26.9 mm, vias 0 -> 1
- net /SDA: track 25.8 -> 50.6 mm, vias 2 -> 3
- net /GPIO3: track 0.00 -> 22.4 mm, vias 0 -> 1
- net /GPIO19: track 0.00 -> 21.2 mm, vias 0 -> 1
- net /GPIO21: track 0.00 -> 21.2 mm, vias 0 -> 1
- net /GPIO8: track 0.00 -> 20.6 mm
- net /GPIO5: track 0.00 -> 20.6 mm, vias 0 -> 1
- net /GPIO20: track 0.00 -> 20.4 mm, vias 0 -> 1
- net /GPIO10: track 0.00 -> 19.7 mm, vias 0 -> 1
- net /GPIO6: track 0.00 -> 19.2 mm
- net /GPIO13: track 0.00 -> 19.1 mm, vias 0 -> 1
- net /GPIO11: track 0.00 -> 18.1 mm, vias 0 -> 1
- net /GPIO7: track 0.00 -> 17.7 mm
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- added copper zone on In4.Cu, net GND
Other:
- copper layers 4 -> 6
