File: PCB/psocpcb_v2/psocpcb.kicad_sch (KiCad schematic)
At the start: 49 parts, among them J1 Conn_01x05, J2 Conn_01x02_Pin, J5 Conn_01x04_Pin, J7 Conn_01x06_Pin, Q1 Si2337DS, U2 AP7365-WG-7, U3 AP2331SA-7, U4 SIP32408DNP-T1-GE4, U5 TXS0102DCUR, U6 AP7365-WG-7, U7 CYBLE-416045-02, Y1 ECS-.327-12.5-34B-TR

Commit message: R3
Parts:
- U7: footprint RASPBERRYPI-ZERO:RASPBERRYPI-ZERO_RPI-ZERO_1_1 -> CYBLE-416045-02:XCVR_CYBLE-416045-02
Connections:
- net SCL: now also A1.13 (GPIO27/GEN2)
- net SDA: now also A1.15 (GPIO22/GEN3)
- net GPIO3: now reaches U7.13 (P10.0)
- net GPIO3: now also A1.16 (GEN4/GPIO23)
- net GPIO4: now reaches U7.14 (P9.4)
- net GPIO4: now also A1.17 (3V3[2])
- net GPIO5: now reaches U7.16 (VREF)
- net GPIO5: now also A1.18 (GEN5/GPIO24)
- net GPIO6: now reaches U7.19 (P9.5)
- net GPIO6: now also A1.19 (GPIO10/MOSI)
- net GPIO1: now reaches U7.2 (P0.5)
- net GPIO1: now also A1.11 (GPIO17/GEN0)
- net GPIO7: now reaches U7.20 (P9.6)
- net GPIO7: now also A1.21 (GPIO9/MISO)
- net GPIO8: now reaches U7.21 (P9.2)
- net GPIO8: now also A1.22 (GEN/6GPIO25)
- net GPIO9: now reaches U7.22 (P7.2)
- net GPIO9: now also A1.23 (GPIO11/SCLK)
- net GPIO10: now reaches U7.23 (P7.1)
- net GPIO10: now also A1.24 (~{CE0}/GPIO8)
- net GPIO11: now reaches U7.24 (P6.4)
- net GPIO11: now also A1.26 (~{CE1}/~{GPIO7})
- net GPIO12: now reaches U7.25 (P5.4)
- net GPIO12: now also A1.27 (ID_SD)
- net GPIO13: now reaches U7.28 (P6.2)
- net GPIO13: now also A1.28 (ID_SC)
- net GPIO14: now reaches U7.29 (P6.5)
- net GPIO14: now also A1.29 (GPIO5)
- net GPIO15: now reaches U7.31 (P7.7)
- net GPIO15: now also A1.40 (GPIO21)
- net GPIO16: now reaches U7.32 (P5.6)
- net GPIO16: now also A1.37 (GPIO26)
- net GPIO17: now reaches U7.34 (P12.6)
- net GPIO17: now also A1.38 (GPIO20)
- net GPIO18: now reaches U7.35 (P12.7)
- net GPIO18: now also A1.35 (GPIO19)
- net GPIO19: now reaches U7.36 (P5.5)
- net GPIO19: now also A1.36 (GPIO16)
- net GPIO20: now reaches U7.37 (P5.3)
- net GPIO20: now also A1.33 (GPIO13)
- net GPIO21: now reaches U7.38 (P5.2)
- net GPIO21: now also A1.31 (GPIO6)
- net GPIO22: now reaches U7.41 (P0.4)
- net GPIO22: now also A1.32 (GPIO12)
- net GPIO2: now reaches U7.9 (P9.3)
- net GPIO2: now also A1.12 (GPIO18)
- no-connect marks 49 -> 3
